File: Training_Robot_Shawn/Training_Robot.kicad_sch (KiCad schematic)
At the start: 31 parts, among them J1 Conn_01x04_Pin, J2 Conn_01x04_Pin, J3 Conn_01x04_Pin, J4 Conn_01x02_Pin, J5 Conn_01x02_Pin, J6 Conn_01x08_Socket, M1 FrontL, M2 FrontR, M3 BackL, M4 BackR, SW1 SW_SPDT_312, U3 ESP32-S3-DevKitC

Commit message: flip fuse footprint, connect esp 5v/gnd pins to board, remove buck converter
Parts:
- removed SW1: SW_SPDT_312, Button_Switch_THT:SW_Slide_SPDT_Straight_CK_OS102011MS2Q, symbol Switch:SW_SPDT_312
- removed U4: (no value), MARS Custom Footprints:MP1495 Buck Converter, symbol MARS Custom Symbols:Generic_Converter
- H1, H2, H3, H4: footprint MountingHole:MountingHole_4.5mm -> MountingHole:MountingHole_6.5mm
Connections:
- net STBY is gone; now on net +3V3: D1.2 (A), U1.4 (STBY), U2.4 (STBY)
- net +12V: now also J5.1 (Pin_1)
- net +5V: now also U3.21 (5V); no longer J5.1 (Pin_1)
- net GND: now also U3.22 (GND), U3.23 (GND), U3.24 (GND), U3.44 (GND)
- no-connect marks 28 -> 26
